Commit message: fixed some issues with xacro file

File: src/simple_robot_description/models/arm_1dof/arm_1dof.urdf (robot description, URDF)
Before this commit: robot arm_1dof, 0 links, 0 joints
Links:
- added link link_0, mass 10; collision box size=0.4 0.4 0.1; visual box size=0.4 0.4 0.1
- added link link_1, mass 10; collision box size=0.1 0.1 0.2; visual box size=0.1 0.1 0.2
- added link link_2, mass 10; collision box size=0.4 0.1 0.1; visual box size=0.4 0.1 0.1
- added link link_3, mass 10; collision box size=0.4 0.1 0.1; visual box size=0.4 0.1 0.1
- added link top_link, mass 0.1; collision box size=0.1 0.1 0.4; visual box size=0.1 0.1 0.4
Joints:
- added joint joint1: type revolute, parent link_3, child top_link, origin xyz=0.05 0 0.2 rpy=0 0 0, axis 1 0 0, limit lower=-1.57 upper=1.57 effort=100.0 velocity=1.0
- added joint joint_link0_link1: type revolute, parent link_0, child link_1, origin xyz=0.0 0 0.05 rpy=0 0 0, axis 0 0 1, limit lower=-1.57 upper=1.57 effort=100.0 velocity=1.0
- added joint joint_link1_link2: type revolute, parent link_1, child link_2, origin xyz=0.05 0 0.15 rpy=0 1.57057 0, axis 0 0 1, limit lower=-1.57 upper=1.57 effort=100.0 velocity=1.0
- added joint joint_link2_link3: type revolute, parent link_2, child link_3, origin xyz=-0.35 0 0.0 rpy=0 0 0, axis 0 0 1, limit lower=-1.57 upper=1.57 effort=100.0 velocity=1.0

File: src/simple_robot_description/models/arm_1dof/arm_1dof.xacro (robot description, xacro)
@@ -1,5 +1,5 @@
 <?xml version="1.0"?>
 <robot name="arm_1dof" xmlns:xacro="http://www.ros.org/wiki/xacro">
-    <!-- <xacro:include filename="joints.xacro" />
+    <xacro:include filename="joints.xacro" />
     <material name="Black">
         <color rgba="0.0 0.0 0.0 1.0" />
@@ -11,9 +11,9 @@
         <color rgba="1.0 1.0 1.0 1.0" />
     </material>
-    <link name="bottom_link">
+    <link name="link_0">
         <visual>
             <origin rpy="0 0 0" xyz="0 0 0" />
             <geometry>
-                <box size="0.1 0.1 0.5" />
+                <box size="0.4 0.4 0.1" />
             </geometry>
         </visual>
@@ -21,15 +21,99 @@
             <origin rpy="0 0 0" xyz="0 0 0" />
             <geometry>
-                <box size="0.1 0.1 0.5" />
+                <box size="0.4 0.4 0.1" />
             </geometry>
         </collision>
         <inertial>
-            <mass value="100" />
+            <mass value="10" />
             <inertia ixx="0.03" iyy="0.03" izz="0.03" ixy="0.0" ixz="0.0" iyz="0.0" />
         </inertial>
     </link>
-    <gazebo reference="bottom_link">
+    <gazebo reference="link_0">
+        <material>Gazebo/Black</material>
+    </gazebo>
+    <link name="link_1">
+        <visual>
+            <origin rpy="0 0 0" xyz="0 0 0.1" />
+            <geometry>
+                <box size="0.1 0.1 0.2" />
+            </geometry>
+        </visual>
+        <collision>
+            <origin rpy="0 0 0" xyz="0 0 0.1" />
+            <geometry>
+                <box size="0.1 0.1 0.2" />
+            </geometry>
+        </collision>
+        <inertial>
+            <mass value="10" />
+            <inertia ixx="0.03" iyy="0.03" izz="0.03" ixy="0.0" ixz="0.0" iyz="0.0" />
+        </inertial>
+    </link>
+    <gazebo reference="link_1">
         <material>Gazebo/Red</material>
     </gazebo>
+     <joint name="joint_link0_link1" type="revolute" >
+        <origin rpy="0 0 0" xyz="0.0 0 0.05" />
+        <parent link="link_0" />
+        <child link="link_1" />
+        <axis xyz="0 0 1" />
+        <limit effort="100.0" lower="-1.57" upper="1.57" velocity="1.0" />
+    </joint>
+    <link name="link_2">
+        <visual>
+            <origin rpy="0 0 0" xyz="-0.2 0 0.05" />
+            <geometry>
+                <box size="0.4 0.1 0.1" />
+            </geometry>
+        </visual>
+        <collision>
+            <origin rpy="0 0 0" xyz="-0.2 0 0.05" />
+            <geometry>
+                <box size="0.4 0.1 0.1" />
+            </geometry>
+        </collision>
+        <inertial>
+            <mass value="10" />
+            <inertia ixx="0.03" iyy="0.03" izz="0.03" ixy="0.0" ixz="0.0" iyz="0.0" />
+        </inertial>
+    </link>
+    <gazebo reference="link_2">
+        <material>Gazebo/White</material>
+    </gazebo>
+    <joint name="joint_link1_link2" type="revolute" >
+        <origin rpy="0 1.57057 0" xyz="0.05 0 0.15" />
+        <parent link="link_1" />
+        <child link="link_2" />
+        <axis xyz="0 0 1" />
+        <limit effort="100.0" lower="-1.57" upper="1.57" velocity="1.0" />
+    </joint>
+    <link name="link_3">
+        <visual>
+            <origin rpy="0 0 0" xyz="-0.2 0 -0.05" />
+            <geometry>
+                <box size="0.4 0.1 0.1" />
+            </geometry>
+        </visual>
+        <collision>
+            <origin rpy="0 0 0" xyz="-0.2 0 -0.05" />
+            <geometry>
+                <box size="0.4 0.1 0.1" />
+            </geometry>
+        </collision>
+        <inertial>
+            <mass value="10" />
+            <inertia ixx="0.03" iyy="0.03" izz="0.03" ixy="0.0" ixz="0.0" iyz="0.0" />
+        </inertial>
+    </link>
+    <gazebo reference="link_3">
+        <material>Gazebo/Red</material>
+    </gazebo>
+    <joint name="joint_link2_link3" type="revolute" >
+        <origin rpy="0 0 0" xyz="-0.35 0 0.0" />
+        <parent link="link_2" />
+        <child link="link_3" />
+        <axis xyz="0 0 1" />
+        <limit effort="100.0" lower="-1.57" upper="1.57" velocity="1.0" />
+    </joint>
     <link name="top_link">
         <visual>
@@ -55,9 +139,9 @@
     <joint name="joint1" type="revolute" >
         <origin rpy="0 0 0" xyz="0.05 0 0.2" />
-        <parent link="bottom_link" />
+        <parent link="link_3" />
         <child link="top_link" />
         <axis xyz="1 0 0" />
         <limit effort="100.0" lower="-1.57" upper="1.57" velocity="1.0" />
     </joint>
-    <xacro:config_ctr_gazebo />  -->
+    <xacro:config_ctr_gazebo />
 </robot>

File: src/simple_robot_description/models/arm_1dof/joints.xacro (robot description, xacro)
@@ -4,5 +4,4 @@
         <!-- I need this for ROS2 control -->
         <!-- I create this file, it was NOT available in the original Doosan repo -->
-<!--
         <ros2_control name="GazeboSystem" type="system">
             <hardware>
@@ -25,5 +24,5 @@
                 <parameters>$(find simple_robot_description)/config/arm_1dof.yaml</parameters>
             </plugin>
-        </gazebo> -->
+        </gazebo>
     </xacro:macro>
 </robot>
