Commit message: update naming issues

File: src/simple_robot_description/models/arm_3dof/arm_3dof.urdf (robot description, URDF)
Before this commit: robot arm_1dof, 5 links, 4 joints
Links:
- removed link top_link
Joints:
- removed joint joint1

File: src/simple_robot_description/models/arm_3dof/arm_3dof.xacro (robot description, xacro)
@@ -1,4 +1,4 @@
 <?xml version="1.0"?>
-<robot name="arm_1dof" xmlns:xacro="http://www.ros.org/wiki/xacro">
+<robot name="arm_3dof" xmlns:xacro="http://www.ros.org/wiki/xacro">
     <xacro:include filename="joints.xacro" />
     <material name="Black">
@@ -11,4 +11,5 @@
         <color rgba="1.0 1.0 1.0 1.0" />
     </material>
+    <!-- Link 0 -->
     <link name="link_0">
         <visual>
@@ -32,4 +33,5 @@
         <material>Gazebo/Black</material>
     </gazebo>
+    <!-- Link 1 -->
     <link name="link_1">
         <visual>
@@ -53,5 +55,5 @@
         <material>Gazebo/Red</material>
     </gazebo>
-     <joint name="joint_link0_link1" type="revolute" >
+    <joint name="joint_link0_link1" type="revolute" >
         <origin rpy="0 0 0" xyz="0.0 0 0.05" />
         <parent link="link_0" />
@@ -60,4 +62,5 @@
         <limit effort="100.0" lower="-1.57" upper="1.57" velocity="1.0" />
     </joint>
+    <!-- Link 2 -->
     <link name="link_2">
         <visual>
@@ -88,4 +91,5 @@
         <limit effort="100.0" lower="-1.57" upper="1.57" velocity="1.0" />
     </joint>
+    <!-- Link 3 -->
     <link name="link_3">
         <visual>
@@ -116,32 +120,4 @@
         <limit effort="100.0" lower="-1.57" upper="1.57" velocity="1.0" />
     </joint>
-    <link name="top_link">
-        <visual>
-            <origin rpy="0 0 0" xyz="0.05 0 0.2" />
-            <geometry>
-                <box size="0.1 0.1 0.4" />
-            </geometry>
-        </visual>
-        <collision>
-            <origin rpy="0 0 0" xyz="0.05 0 0.2" />
-            <geometry>
-                <box size="0.1 0.1 0.4" />
-            </geometry>
-        </collision>
-        <inertial>
-            <mass value="0.1" />
-            <inertia ixx="0.03" iyy="0.03" izz="0.03" ixy="0.0" ixz="0.0" iyz="0.0" />
-        </inertial>
-    </link>
-    <gazebo reference="top_link">
-        <material>Gazebo/White</material>
-    </gazebo>
-    <joint name="joint1" type="revolute" >
-        <origin rpy="0 0 0" xyz="0.05 0 0.2" />
-        <parent link="link_3" />
-        <child link="top_link" />
-        <axis xyz="1 0 0" />
-        <limit effort="100.0" lower="-1.57" upper="1.57" velocity="1.0" />
-    </joint>
     <xacro:config_ctr_gazebo />
 </robot>

File: src/simple_robot_description/models/arm_3dof/joints.xacro (robot description, xacro)
@@ -22,5 +22,5 @@
                 <!--<robot_sim_type>gazebo_ros2_control/DefaultRobotHWSim</robot_sim_type> -->
                 <robot_sim_type>gazebo_ros2_control/GazeboSystem</robot_sim_type>
-                <parameters>$(find simple_robot_description)/config/arm_1dof.yaml</parameters>
+                <parameters>$(find simple_robot_description)/config/arm_3dof.yaml</parameters>
             </plugin>
         </gazebo>
